Commit message: Day 2 complete: Gazebo Harmonic diff drive with ros_gz_bridge

File: src/robot_description/urdf/robot.urdf.xacro (robot description, xacro)
@@ -1,4 +1,5 @@
 <?xml version="1.0"?>
 <robot name="mobile_robot">
+  <!-- Base link -->
   <link name="base_link">
     <visual>
@@ -19,3 +20,73 @@
     </inertial>
   </link>
+  <!-- Left wheel -->
+  <link name="left_wheel">
+    <visual>
+      <geometry>
+        <cylinder radius="0.05" length="0.02"/>
+      </geometry>
+      <origin rpy="1.5708 0 0"/>
+    </visual>
+    <collision>
+      <geometry>
+        <cylinder radius="0.05" length="0.02"/>
+      </geometry>
+      <origin rpy="1.5708 0 0"/>
+    </collision>
+    <inertial>
+      <mass value="0.5"/>
+      <inertia ixx="0.001" iyy="0.001" izz="0.001"
+               ixy="0.0" ixz="0.0" iyz="0.0"/>
+    </inertial>
+  </link>
+  <!-- Right wheel -->
+  <link name="right_wheel">
+    <visual>
+      <geometry>
+        <cylinder radius="0.05" length="0.02"/>
+      </geometry>
+      <origin rpy="1.5708 0 0"/>
+    </visual>
+    <collision>
+      <geometry>
+        <cylinder radius="0.05" length="0.02"/>
+      </geometry>
+      <origin rpy="1.5708 0 0"/>
+    </collision>
+    <inertial>
+      <mass value="0.5"/>
+      <inertia ixx="0.001" iyy="0.001" izz="0.001"
+               ixy="0.0" ixz="0.0" iyz="0.0"/>
+    </inertial>
+  </link>
+  <!-- Left wheel joint -->
+  <joint name="left_wheel_joint" type="continuous">
+    <parent link="base_link"/>
+    <child link="left_wheel"/>
+    <origin xyz="0 0.15 -0.05"/>
+    <axis xyz="0 1 0"/>
+  </joint>
+  <!-- Right wheel joint -->
+  <joint name="right_wheel_joint" type="continuous">
+    <parent link="base_link"/>
+    <child link="right_wheel"/>
+    <origin xyz="0 -0.15 -0.05"/>
+    <axis xyz="0 1 0"/>
+  </joint>
+    <!-- Gazebo diff drive plugin -->
+    <!-- Gazebo Harmonic diff drive system -->
+  <gazebo>
+    <plugin filename="gz-sim-diff-drive-system"
+            name="gz::sim::systems::DiffDrive">
+      <left_joint>left_wheel_joint</left_joint>
+      <right_joint>right_wheel_joint</right_joint>
+      <wheel_separation>0.30</wheel_separation>
+      <wheel_radius>0.05</wheel_radius>
+      <odom_publish_frequency>50</odom_publish_frequency>
+      <topic>cmd_vel</topic>
+      <odom_topic>odom</odom_topic>
+      <frame_id>odom</frame_id>
+      <child_frame_id>base_link</child_frame_id>
+    </plugin>
+  </gazebo>
 </robot>

Commit message: Day 3 complete: Differential drive robot with LiDAR in Gazebo Harmonic

File: src/robot_description/urdf/robot.urdf.xacro (robot description, xacro)
@@ -1,5 +1,4 @@
 <?xml version="1.0"?>
 <robot name="mobile_robot">
-  <!-- Base link -->
   <link name="base_link">
     <visual>
@@ -15,10 +14,8 @@
     <inertial>
       <mass value="5.0"/>
-      <origin xyz="0 0 0"/>
       <inertia ixx="0.1" iyy="0.1" izz="0.1"
                ixy="0.0" ixz="0.0" iyz="0.0"/>
     </inertial>
   </link>
-  <!-- Left wheel -->
   <link name="left_wheel">
     <visual>
@@ -40,5 +37,4 @@
     </inertial>
   </link>
-  <!-- Right wheel -->
   <link name="right_wheel">
     <visual>
@@ -54,5 +50,5 @@
       <origin rpy="1.5708 0 0"/>
     </collision>
-    <inertial>
+     <inertial>
       <mass value="0.5"/>
       <inertia ixx="0.001" iyy="0.001" izz="0.001"
@@ -60,5 +56,16 @@
     </inertial>
   </link>
-  <!-- Left wheel joint -->
+  <link name="lidar_link">
+    <visual>
+      <geometry>
+        <cylinder radius="0.04" length="0.05"/>
+      </geometry>
+    </visual>
+    <collision>
+      <geometry>
+        <cylinder radius="0.04" length="0.05"/>
+      </geometry>
+    </collision>
+  </link>
   <joint name="left_wheel_joint" type="continuous">
     <parent link="base_link"/>
@@ -67,5 +74,4 @@
     <axis xyz="0 1 0"/>
   </joint>
-  <!-- Right wheel joint -->
   <joint name="right_wheel_joint" type="continuous">
     <parent link="base_link"/>
@@ -74,6 +80,9 @@
     <axis xyz="0 1 0"/>
   </joint>
-    <!-- Gazebo diff drive plugin -->
-    <!-- Gazebo Harmonic diff drive system -->
+  <joint name="lidar_joint" type="fixed">
+    <parent link="base_link"/>
+    <child link="lidar_link"/>
+    <origin xyz="0.2 0 0.1"/>
+  </joint>
   <gazebo>
     <plugin filename="gz-sim-diff-drive-system"
@@ -83,5 +92,4 @@
       <wheel_separation>0.30</wheel_separation>
       <wheel_radius>0.05</wheel_radius>
-      <odom_publish_frequency>50</odom_publish_frequency>
       <topic>cmd_vel</topic>
       <odom_topic>odom</odom_topic>
@@ -90,3 +98,23 @@
     </plugin>
   </gazebo>
+  <gazebo reference="lidar_link">
+    <sensor name="lidar" type="gpu_lidar">
+      <update_rate>10</update_rate>
+      <lidar>
+        <scan>
+          <horizontal>
+            <samples>720</samples>
+            <min_angle>-1.5708</min_angle>
+            <max_angle>1.5708</max_angle>
+          </horizontal>
+        </scan>
+        <range>
+          <min>0.12</min>
+          <max>10.0</max>
+        </range>
+      </lidar>
+      <visualize>true</visualize>
+      <topic>scan</topic>
+    </sensor>
+  </gazebo>
 </robot>
